File: triumph-power/triumph_power.kicad_pcb (KiCad board)
At the start: 2 copper layers, 53.3 x 33 mm, 22 parts, among them J1 JST_XH_vert_01x04, J2 JST_XH_vert_01x04, U1 RS-1212D

Commit message: Make cosmetic edits
Parts:
- added G***: LOGO, triumph-logos:ruddock-crest-small, B.Cu at (142.2, 109.2)
